File: idock_pcb0-1.kicad_pcb (KiCad board)
At the start: 2 copper layers, 99.7 x 78.1 mm, 24 parts, among them J1 Barrel_Jack_Switch, J2 dock, J3 POWERLED, J4 PJRAN2X1U02, J5 Bluetooth Module, Q1 BC548, SW1 Reset, U1 ATmega32A-PU, Y1 8mhz

Commit message: release pcb to jclpcb
Parts:
- moved TP5 39.7 mm to (193.7, 78.7)
- moved D1 8.25 mm to (175.7, 106.7)
- moved R2 7.75 mm to (181.4, 110.5)
- moved R4 7.66 mm to (188.0, 110.5)
- moved C1 6.38 mm to (166.8, 113.5)
- moved C2 6.38 mm to (163.3, 113.5)
- moved TP3 6.38 mm to (144.8, 107.3)
- moved Y1 6.38 mm to (167.3, 108.2)
- moved R1 6.38 mm to (156.2, 118.7)
- moved SW1 6.38 mm to (156.2, 111.6)
Routing:
- net Net-(J5-Pad4): track 36.7 -> 28.3 mm
- net Net-(R2-Pad2): track 11.8 -> 3.96 mm
- net +5V: track 141.3 -> 134.7 mm
- net Net-(C2-Pad1): track 22.0 -> 15.4 mm
- net Net-(R1-Pad2): track 39.6 -> 33.2 mm
- net Net-(C1-Pad1): track 22.2 -> 16.1 mm
- net Net-(J2-Pad4): track 88.4 -> 84.6 mm
- net Net-(J2-Pad5): track 87.8 -> 87.2 mm
Other:
- board text added: "2n2222"
- board text added: "AUDIO OUT"
- board text added: "Designed by RattaMayhorka"
- board text added: "GND"
- board text added: "IPOD IN"
- board text added: "POWER"
- board text added: "VCC"
